Commit message: update simulator

File: 3D/urdf/cubli.urdf (robot description, URDF)
Before this commit: robot cubli, 1 links, 0 joints
Links:
- added link flywheel_pitch; collision mesh filename=mesh/flywheel.stl; visual mesh filename=mesh/flywheel.stl
- link base_link: geometry collision mesh filename=mesh/body.stl; visual mesh filename=mesh/body.stl
Joints:
- added joint flywheel_pitch_motor: type revolute, parent base_link, child flywheel_pitch, limit effort=100 velocity=1000.0

Commit message: update cubli

File: 3D/urdf/cubli.urdf (robot description, URDF)
Before this commit: robot cubli, 2 links, 1 joints
Links:
- removed link flywheel_pitch
- added link flywheel_yaw; collision mesh filename=mesh/flywheel.stl; visual mesh filename=mesh/flywheel.stl
Joints:
- removed joint flywheel_pitch_motor
- added joint flywheel_yaw_motor: type revolute, parent base_link, child flywheel_yaw, axis 1 0 0, limit effort=100 velocity=1000.0
